File: hw/ETH_module.brd (EAGLE design)
At the start: 50 x 45 mm, 58 parts, among them J1 R2P_BUS-VERTICAL, J2 R2P_BUS-VERTICAL, J3 MICROSD-3300060P1, J4 MICRO-USB-5P-340015001, U1 STM32F407VG, U2 CM1624, X1 RJ45-MAG-RB1-125BAG1A

Commit message: Layout complete
Parts:
- removed R3: 100k, r2p_rcl:R0603
- added C27: (no value), rcl:B/3528-21R
- added D1: MBR0520LT, diode:SOD123
- added X5: 53047-04, con-molex:53047-04
- OSC1: value 8MHz -> 24Mhz
- moved C10 45.6 mm to (18.0, 6.30), turned to 180 degrees
- moved J4 43.7 mm to (43.0, 42.5), turned to 180 degrees
- moved C19 40.5 mm to (34.7, 23.4), turned to 90 degrees
- moved C21 40.2 mm to (22.6, 23.6), turned to 90 degrees
- moved C20 39.0 mm to (40.5, 12.0)
- moved C18 35.4 mm to (34.8, 2.70), turned to 180 degrees
- moved C3 35.1 mm to (40.5, 17.4)
- moved C23 31.5 mm to (16.7, 22.5), turned to 0 degrees
- moved R6 29.4 mm to (33.3, 23.4), turned to 270 degrees
- moved C11 29.0 mm to (40.5, 16.0), turned to 180 degrees
- moved X1 27.0 mm to (11.5, 36.1)
- moved C14 26.9 mm to (25.5, 28.2), turned to 270 degrees
- moved C15 23.3 mm to (23.9, 28.1), turned to 270 degrees
- moved LED2 21.3 mm to (37.9, 36.6)
- moved R8 20.5 mm to (41.0, 36.5), turned to 90 degrees
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Connections:
- removed net N$3: OSC1.1, R3.2
- removed net SD_CLK: U2.14
- removed net SD_CMD: U2.11
- removed net SD_DATA0: U2.15
- removed net SD_DATA1: U2.16
- removed net SD_DATA2: U2.9
- removed net SD_DATA3: U2.10
- removed net USB_ID: U1.69
- removed net USB_N: R11.1
- removed net USB_P: R14.1
- new net SDIO_CK: U1.80, U2.14
- new net SDIO_CMD: U1.83, U2.11
- new net SDIO_D0: U1.65, U2.15
- new net SDIO_D1: U1.66, U2.16
- new net SDIO_D2: U1.78, U2.9
- new net SDIO_D3: U1.79, U2.10
- net +3V3: now also OSC1.1, X5.1; no longer R3.1
- net +VBUS: now also C27.+, D1.C
- net ETH_PHYAD0: now also U1.60; no longer U1.63
- net ETH_RST: now also U1.57; no longer U1.64
- net GND: now also C27.-, X1.8, X5.2
- net LED1: now also U1.5; no longer U1.78
- net SD_LED: now also U1.29
- net UART_RX: now also X5.4
- net UART_TX: now also X5.3
- net USB_DM: now also R11.1
- net USB_DP: now also R14.1
- net USB_VBUS: now also D1.A; no longer U1.68
Routing:
- net +3V3: track 51.7 -> 200.5 mm, vias 4 -> 18
- net USB_DP: track 0.00 -> 41.1 mm, vias 0 -> 2
- net USB_DM: track 0.00 -> 40.7 mm, vias 0 -> 2
- net +VBUS: track 7.26 -> 44.4 mm
- net ETH_RMII_RXD1: track 0.00 -> 30.9 mm, vias 0 -> 2
- net ETH_RMII_RXD0: track 0.00 -> 30.2 mm, vias 0 -> 2
- net UART_TX: track 0.00 -> 27.0 mm, vias 0 -> 1
- net ETH_RMII_MDIO: track 3.16 -> 29.5 mm, vias 0 -> 2
- net SDIO_CK: track 0.00 -> 25.9 mm, vias 0 -> 2
- net UART_RX: track 0.00 -> 25.8 mm, vias 0 -> 1
- net SDIO_D2: track 0.00 -> 25.7 mm, vias 0 -> 2
- net 3V3_ETH: track 5.96 -> 31.5 mm, vias 2 -> 3
- net SDIO_D3: track 0.00 -> 25.4 mm, vias 0 -> 2
- net SDIO_CMD: track 0.00 -> 25.1 mm, vias 0 -> 2
- net ETH_RMII_CRS_DV: track 0.00 -> 25.0 mm, vias 0 -> 2
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
Commit message: Fixed silkscreen
Connections:
- net GND: now also X1.10, X1.9
Other:
- board text added: "ETH module v1.0 (2015/02)"
- board text added: "SD"
Changed lines of the file:
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@@
 <layers>
 <layer number="1" name="Top" color="4" fill="1" visible="yes" active="yes"/>
-<layer number="16" name="Bottom" color="1" fill="1" visible="no" active="yes"/>
+<layer number="16" name="Bottom" color="1" fill="1" visible="yes" active="yes"/>
 <layer number="17" name="Pads" color="2" fill="1" visible="yes" active="yes"/>
 <layer number="18" name="Vias" color="2" fill="1" visible="yes" active="yes"/>
@@
 <wire x1="6.55" y1="8" x2="6.55" y2="8.8" width="0.2" layer="41"/>
 <wire x1="6.55" y1="8.8" x2="7.45" y2="8.8" width="0.2" layer="41"/>
+<text x="4" y="6" size="1.5" layer="200" rot="MR90">ETH module
+v1.0 (2015/02)</text>
+<text x="38" y="34.5" size="1" layer="48" font="vector" rot="R90" align="center-right">SD</text>
 </plain>
 <attributes>
@@
 <via x="0.9" y="43.4" extent="1-16" drill="0.3"/>
 <via x="1.6" y="44.1" extent="1-16" drill="0.3"/>
+<contactref element="X1" pad="9"/>
+<contactref element="X1" pad="10"/>
 </signal>
 <signal name="+VBUS">
@@
 </board>
 </drawing>
+<compatibility>
+<note version="6.3" minversion="6.2.2" severity="warning">
+Since Version 6.2.2 text objects can contain more than one line,
+which will not be processed correctly with this version.
+</note>
+</compatibility>
 </eagle>
