File: hw/ETH_module.sch (EAGLE design)
At the start: 58 parts, among them J1 R2P_BUS-VERTICAL, J2 R2P_BUS-VERTICAL, J3 MICROSD-3300060P1, J4 MICRO-USB-5P-340015001, U1 STM32F407VG, U2 CM1624, X1 RJ45-MAG-RB1-125BAG1A

Commit message: Layout complete
Parts:
- removed R3: 100k, r2p_rcl:R0603
- added C27: (no value), rcl:CPOL-EUB/3528-21R
- added D1: MBR0520LT, diode:MBR0520LT
- added X5: 53047-04, con-molex:53047-04
- OSC1: value 8MHz -> 24Mhz
Connections:
- removed net N$3: OSC1.TRI, R3.2
- removed net SD_CLK: U2.CLK
- removed net SD_CMD: U2.CMD
- removed net SD_DATA0: U2.DATA0
- removed net SD_DATA1: U2.DATA1
- removed net SD_DATA2: U2.DATA2
- removed net SD_DATA3: U2.DATA3
- removed net USB_ID: U1IO.PA10
- removed net USB_N: R11.1
- removed net USB_P: R14.1
- new net SDIO_CK: U1IO.PC12, U2.CLK
- new net SDIO_CMD: U1IO.PD2, U2.CMD
- new net SDIO_D0: U1IO.PC8, U2.DATA0
- new net SDIO_D1: U1IO.PC9, U2.DATA1
- new net SDIO_D2: U1IO.PC10, U2.DATA2
- new net SDIO_D3: U1IO.PC11, U2.DATA3
- net +3V3: now also OSC1.TRI, X5-1.S; no longer R3.1
- net +VBUS: now also C27.+, D1.C
- net ETH_PHYAD0: now also U1IO.PD13; no longer U1IO.PC6
- net ETH_RST: now also U1IO.PD10; no longer U1IO.PC7
- net GND: now also C27.-, X1.8, X5-2.S
- net LED1: now also U1IO.PE6; no longer U1IO.PC10
- net SD_LED: now also U1IO.PA4
- net UART_RX: now also X5-4.S
- net UART_TX: now also X5-3.S
- net USB_DM: now also R11.1
- net USB_DP: now also R14.1
- net USB_VBUS: now also D1.A; no longer U1IO.PA9
Other:
- note added: "POWER ORING"
- note added: "SHIELD DA CONNETTERE!!!"

Commit message: Fixed silkscreen
Connections:
- net GND: now also X1.SHLD1, X1.SHLD2
Other:
- note removed: "SHIELD DA CONNETTERE!!!"
Changed lines of the file:
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@@
 <part name="GND52" library="supply" deviceset="GND" device=""/>
 <part name="C27" library="rcl" deviceset="CPOL-EU" device="B/3528-21R"/>
+<part name="GND53" library="supply" deviceset="GND" device=""/>
 </parts>
 <sheets>
@@
 <wire x1="855.98" y1="375.92" x2="855.98" y2="426.72" width="0.1524" layer="94"/>
 <text x="858.52" y="421.64" size="2.54" layer="94">USB INTERFACE</text>
-<text x="769.62" y="203.2" size="5.08" layer="90">SHIELD DA CONNETTERE!!!</text>
 <wire x1="855.98" y1="515.62" x2="990.6" y2="515.62" width="0.1524" layer="94"/>
 <wire x1="990.6" y1="515.62" x2="990.6" y2="436.88" width="0.1524" layer="94"/>
@@
 <instance part="GND52" gate="1" x="967.74" y="462.28"/>
 <instance part="C27" gate="G$1" x="967.74" y="469.9"/>
+<instance part="GND53" gate="1" x="795.02" y="264.16" rot="R270"/>
 </instances>
 <busses>
@@
 <pinref part="C27" gate="G$1" pin="-"/>
 </segment>
+<segment>
+<pinref part="X1" gate="-1" pin="SHLD1"/>
+<wire x1="802.64" y1="261.62" x2="800.1" y2="261.62" width="0.1524" layer="91"/>
+<wire x1="800.1" y1="261.62" x2="800.1" y2="264.16" width="0.1524" layer="91"/>
+<pinref part="GND53" gate="1" pin="GND"/>
+<wire x1="800.1" y1="264.16" x2="797.56" y2="264.16" width="0.1524" layer="91"/>
+<pinref part="X1" gate="-1" pin="SHLD2"/>
+<wire x1="802.64" y1="264.16" x2="800.1" y2="264.16" width="0.1524" layer="91"/>
+<junction x="800.1" y="264.16"/>
+</segment>
 </net>
